File: Kiosk/SmartIO/hardware/v3.3/SmartIOv3.3.sch (KiCad schematic (older format))
At the start: 52 parts, among them J1 LCD, J10 ADC, J2 DB9, J3 MTN, J4 39910-0102, J6 ISP Hdr, J7 Keypad, J8 Scew terminals, J9 +5V PSU, K1 CB1aH-P-12V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

Commit message: Added mod files for PCB
Parts:
- J8: DigiKeyPN (none) -> ED2739-ND; ManPN (none) -> OSTTE160104
- J9: DigiKeyPN (none) -> ED2740-ND; ManPN (none) -> OSTTE020104
Changed lines of the file:
@@
-EESchema Schematic File Version 2  date Saturday, May 18, 2013 05:48:51 PM
+EESchema Schematic File Version 2  date Friday, May 24, 2013 03:42:45 AM
 LIBS:power
 LIBS:device
@@
 LIBS:contrib
 LIBS:valves
-LIBS:SmartIO-extra-comp
-LIBS:acs754-acs755-acs756
 LIBS:SmartIOv3.3-cache
 EELAYER 27 0
@@
 Sheet 1 1
 Title ""
-Date "18 may 2013"
+Date "24 may 2013"
 Rev ""
 Comp ""
@@
 F 2 "" H 2980 3510 60  0001 C CNN
 F 3 "" H 2980 3510 60  0001 C CNN
+F 4 "ED2739-ND" V 2980 3510 60  0001 C CNN "DigiKeyPN"
+F 5 "OSTTE160104" V 2980 3510 60  0001 C CNN "ManPN"
 	1    2980 3510
 	1    0    0    -1
@@
 F 2 "" H 3610 5430 60  0000 C CNN
 F 3 "" H 3610 5430 60  0000 C CNN
+F 4 "ED2740-ND" V 3610 5430 60  0001 C CNN "DigiKeyPN"
+F 5 "OSTTE020104" V 3610 5430 60  0001 C CNN "ManPN"
 	1    3610 5430
 	0    -1   -1   0

Commit message: Added RC snubber, additional bypass caps for SMD AVR
Parts:
- removed J4: 39910-0102, symbol CONN_2
- added C21, Cb1, Cb3: 0.1uF, symbol C
- added Cb4: 10uF, symbol C
- added J4: 39910-0103, symbol CONN_3
- added R10: 120, symbol R2
- R6: footprint (none) -> POTX
- U2: value ATMEGA164PA-P -> ATMEGA164PA-A; symbol ATMEGA164PA-P -> ATMEGA164PA-A
- renumbered C3 to Cb2
Connections:
- wire segments 80 -> 99
Other:
- note added: "AC/DC RC Snubber\nAC X2-type Cap\n120 Ohm 1/2 W R"
- moved on the sheet: C4, Cb2, FB1, R1, R2

Commit message: Added 5v sw PSU module V78XX-2000
Parts:
- removed J9: +5V PSU, symbol CONN_2
- added C22: 10uF, symbol C
- added C23: 22uF, symbol C
- added U5: V7805-2000, symbol LM7805
Connections:
- wire segments 99 -> 101
Other:
- note added: "12 V Power hold-up\nWith 5 V 2 A Sw. PSU\nV7805-2000"
- note removed: "12 V Power hold-up\nfor 5v PSU"
Changed lines of the file:
@@
 Text GLabel 2630 3110 0    45   Input ~ 0
 DRSN
-Text GLabel 3250 7500 0    45   Input ~ 0
-+5V
-$Comp
-L +5V #PWR016
-U 1 1 5197C70F
-P 3330 7420
-F 0 "#PWR016" H 3330 7510 20  0001 C CNN
-F 1 "+5V" H 3210 7470 49  0000 C CNN
-F 2 "" H 3330 7420 60  0001 C CNN
-F 3 "" H 3330 7420 60  0001 C CNN
-	1    3330 7420
-	1    0    0    -1
-$EndComp
 Text GLabel 2630 3210 0    45   Input ~ 0
 +5V
@@
 GND
 $Comp
-L +12V #PWR017
+L +12V #PWR016
 U 1 1 5197D1F0
 P 2710 5780
-F 0 "#PWR017" H 2710 5730 20  0001 C CNN
+F 0 "#PWR016" H 2710 5730 20  0001 C CNN
 F 1 "+12V" H 2570 5840 49  0000 C CNN
 F 2 "" H 2710 5780 60  0001 C CNN
@@
 Text GLabel 2710 6180 0    45   Input ~ 0
 GND
-$Comp
-L CONN_2 J9
-U 1 1 5197D288
-P 3610 5430
-F 0 "J9" V 3630 5430 40  0000 C CNN
-F 1 "+5V PSU" V 3760 5440 40  0000 C CNN
-F 2 "" H 3610 5430 60  0001 C CNN
-F 3 "" H 3610 5430 60  0001 C CNN
-F 4 "ED2740-ND" V 3610 5430 60  0001 C CNN "DigiKeyPN"
-F 5 "OSTTE020104" V 3610 5430 60  0001 C CNN "ManPN"
-	1    3610 5430
-	0    -1   -1   0
-$EndComp
 Text GLabel 3810 5780 2    45   Input ~ 0
 GND
@@
 Text GLabel 4270 2950 0    45   Input ~ 0
 GND
-Text GLabel 3720 7530 0    45   Input ~ 0
-GND
-$Comp
-L GND #PWR018
+Text GLabel 3420 7530 0    45   Input ~ 0
+GND
+$Comp
+L GND #PWR017
 U 1 1 5197D8A8
-P 3810 7590
-F 0 "#PWR018" H 3810 7590 30  0001 C CNN
-F 1 "GND" H 3810 7520 30  0001 C CNN
-F 2 "" H 3810 7590 60  0001 C CNN
-F 3 "" H 3810 7590 60  0001 C CNN
-	1    3810 7590
-	1    0    0    -1
-$EndComp
-$Comp
-L PWR_FLAG #FLG019
+P 3510 7590
+F 0 "#PWR017" H 3510 7590 30  0001 C CNN
+F 1 "GND" H 3510 7520 30  0001 C CNN
+F 2 "" H 3510 7590 60  0001 C CNN
+F 3 "" H 3510 7590 60  0001 C CNN
+	1    3510 7590
+	1    0    0    -1
+$EndComp
+$Comp
+L PWR_FLAG #FLG018
 U 1 1 5197DD72
-P 3810 7530
-F 0 "#FLG019" H 3810 7625 30  0001 C CNN
-F 1 "PWR_FLAG" H 3810 7710 30  0000 C CNN
-F 2 "" H 3810 7530 60  0001 C CNN
-F 3 "" H 3810 7530 60  0001 C CNN
-	1    3810 7530
-	1    0    0    -1
-$EndComp
+P 3510 7530
+F 0 "#FLG018" H 3510 7625 30  0001 C CNN
+F 1 "PWR_FLAG" H 3510 7710 30  0000 C CNN
+F 2 "" H 3510 7530 60  0001 C CNN
+F 3 "" H 3510 7530 60  0001 C CNN
+	1    3510 7530
+	1    0    0    -1
+$EndComp
+$Comp
+L +12V #PWR019
+U 1 1 5197DE41
+P 3000 7420
+F 0 "#PWR019" H 3000 7370 20  0001 C CNN
+F 1 "+12V" H 2860 7480 49  0000 C CNN
+F 2 "" H 3000 7420 60  0001 C CNN
+F 3 "" H 3000 7420 60  0001 C CNN
+	1    3000 7420
+	1    0    0    -1
+$EndComp
+Text GLabel 2940 7480 0    45   Input ~ 0
++12V
 $Comp
 L PWR_FLAG #FLG020
-U 1 1 5197DE0A
-P 3330 7500
-F 0 "#FLG020" H 3330 7595 30  0001 C CNN
-F 1 "PWR_FLAG" H 3330 7680 30  0000 C CNN
-F 2 "" H 3330 7500 60  0001 C CNN
-F 3 "" H 3330 7500 60  0001 C CNN
-	1    3330 7500
-	-1   0    0    1
-$EndComp
-$Comp
-L +12V #PWR021
-U 1 1 5197DE41
-P 2850 7420
-F 0 "#PWR021" H 2850 7370 20  0001 C CNN
-F 1 "+12V" H 2710 7480 49  0000 C CNN
-F 2 "" H 2850 7420 60  0001 C CNN
-F 3 "" H 2850 7420 60  0001 C CNN
-	1    2850 7420
-	1    0    0    -1
-$EndComp
-Text GLabel 2790 7480 0    45   Input ~ 0
-+12V
-$Comp
-L PWR_FLAG #FLG022
 U 1 1 5197DE4A
-P 2850 7480
-F 0 "#FLG022" H 2850 7575 30  0001 C CNN
-F 1 "PWR_FLAG" H 2850 7660 30  0000 C CNN
-F 2 "" H 2850 7480 60  0001 C CNN
-F 3 "" H 2850 7480 60  0001 C CNN
-	1    2850 7480
-	-1   0    0    1
-$EndComp
-$Comp
-L PWR_FLAG #FLG023
+P 3000 7480
+F 0 "#FLG020" H 3000 7575 30  0001 C CNN
+F 1 "PWR_FLAG" H 3000 7660 30  0000 C CNN
+F 2 "" H 3000 7480 60  0001 C CNN
+F 3 "" H 3000 7480 60  0001 C CNN
+	1    3000 7480
+	-1   0    0    1
+$EndComp
+$Comp
+L PWR_FLAG #FLG021
 U 1 1 5197E383
 P 4670 2950
-F 0 "#FLG023" H 4670 3045 30  0001 C CNN
+F 0 "#FLG021" H 4670 3045 30  0001 C CNN
 F 1 "PWR_FLAG" H 4670 3130 30  0000 C CNN
 F 2 "" H 4670 2950 60  0001 C CNN
@@
 Text Notes 4720 5840 0    60   ~ 0
 Power Relay, Drive (PA7) and Current Sense (PA1)
-Text Notes 2440 5340 0    60   ~ 0
-12 V Power hold-up\nfor 5v PSU
+Text Notes 2440 5060 0    60   ~ 0
+12 V Power hold-up\nWith 5 V 2 A Sw. PSU\nV7805-2000
 Text Notes 8650 4950 0    60   ~ 0
 RS232 for CPU and MSR
@@
 GND
 $Comp
-L PWR_FLAG #FLG024
+L PWR_FLAG #FLG022
 U 1 1 5197F6B0
 P 5810 773
-F 0 "#FLG024" H 5810 868 30  0001 C CNN
+F 0 "#FLG022" H 5810 868 30  0001 C CNN
 F 1 "PWR_FLAG" H 5810 953 30  0000 C CNN
 F 2 "" H 5810 773 60  0001 C CNN
@@
 $EndComp
 $Comp
-L +5V #PWR025
+L +5V #PWR023
 U 1 1 51C092CC
 P 4615 1375
-F 0 "#PWR025" H 4615 1465 20  0001 C CNN
+F 0 "#PWR023" H 4615 1465 20  0001 C CNN
 F 1 "+5V" H 4505 1425 49  0000 C CNN
 F 2 "" H 4615 1375 60  0001 C CNN
@@
 	3410 6980 3810 6980
 Wire Wire Line
-	3110 5780 3510 5780
-Connection ~ 3410 5780
-Wire Wire Line
-	3710 5780 3810 5780
-Wire Wire Line
-	3810 7590 3810 7530
-Wire Wire Line
-	3810 7530 3720 7530
-Wire Wire Line
-	3330 7420 3330 7500
-Wire Wire Line
-	3330 7500 3250 7500
-Wire Wire Line
-	2790 7480 2850 7480
-Wire Wire Line
-	2850 7480 2850 7420
+	3110 5780 3410 5780
+Wire Wire Line
+	3810 5550 3810 5780
+Wire Wire Line
+	3510 7590 3510 7530
+Wire Wire Line
+	3510 7530 3420 7530
+Wire Wire Line
+	2940 7480 3000 7480
+Wire Wire Line
+	3000 7480 3000 7420
 Connection ~ 4450 1950
 Wire Wire Line
@@
 	7450 6350 6410 6350
 Connection ~ 6310 6460
+$Comp
+L LM7805 U5
+U 1 1 51C25E9D
+P 3810 5300
+F 0 "U5" H 3960 5104 60  0000 C CNN
+F 1 "V7805-2000" H 3890 5510 60  0000 C CNN
+F 2 "" H 3810 5300 60  0000 C CNN
+F 3 "" H 3810 5300 60  0000 C CNN
+	1    3810 5300
+	1    0    0    -1
+$EndComp
+$Comp
+L C C23
+U 1 1 51C25ECB
+P 4210 5450
+F 0 "C23" V 4230 5570 50  0000 C TNN
+F 1 "22uF" V 4250 5260 39  0000 L CNN
+F 2 "" H 4210 5450 60  0001 C CNN
+F 3 "" H 4210 5450 60  0001 C CNN
+	1    4210 5450
+	-1   0    0    1
+$EndComp
+$Comp
+L C C22
+U 1 1 51C25ED1
+P 3410 5450
+F 0 "C22" V 3430 5570 50  0000 C TNN
+F 1 "10uF" V 3450 5260 39  0000 L CNN
+F 2 "" H 3410 5450 60  0001 C CNN
+F 3 "" H 3410 5450 60  0001 C CNN
+	1    3410 5450
+	-1   0    0    1
+$EndComp
+Wire Wire Line
+	3410 5650 4210 5650
+Connection ~ 3810 5650
+Text GLabel 4300 5250 2    45   Input ~ 0
++5V
+Wire Wire Line
+	4300 5250 4210 5250
+Wire Wire Line
+	3410 5250 3250 5250
+Wire Wire Line
+	3250 5250 3250 5780
+Connection ~ 3250 5780
 $EndSCHEMATC

Commit message: Fixed snubber and power terminal connections
Parts:
- C10, C11, C7, C8, C9: symbol CP1 -> C
- J4: symbol CONN_3 -> TERM-3
- renumbered C4 to Cb5, C2 to Cb6
Connections:
- wire segments 101 -> 100
Other:
- note added: "12 V Power hold-up\nWith 5V 2A Sw. PSU\nV7805-2000"
- note added: "LCD Header, BL, cntrst (Port C)"
- note added: "NB: NT/GND pin\nused for EMI return ONLY\nNOT power return!"
- note added: "Power Relay, Drive (PA7) and Current Sense (PA1)\nIsolated PWR, NT/GND. 12VDC/120VAC."
- note removed: "12 V Power hold-up\nWith 5 V 2 A Sw. PSU\nV7805-2000"
- note removed: "LCD Header & BL control (Port C)"
- note removed: "Power Relay, Drive (PA7) and Current Sense (PA1)"
- moved on the sheet: C21, Cb5, Cb6, D1, K1, R10, R5, U1, U3

Commit message: Added OLinuXino-MICRO header, made a pre-module-packing version of the board
Parts:
- added J11: TTL UART, symbol TERM-5
- added Q5, Q6: BSS138K, symbol MOSFET_N
- added R11, R12, R13, R14: 10k, symbol R2
- J1: symbol CONN_8X2 -> TERM-8X2
- J3: symbol CONN_3 -> TERM-3
- J4: symbol TERM-3 -> SW-PWR-3
- J6: symbol CONN_3X2 -> TERM-3X2
- J7: symbol CONN_8 -> TERM-8
- J8: symbol CONN_16 -> TERM-16
Connections:
- net labels added: TTL-Rx, TTL-Tx, V-TTL
- wire segments 100 -> 102
Other:
- note added: "TTL UART Voltage Conv."
- moved on the sheet: C1, C12, C13, C14, C15, C16, C17, C18, C21, C5, Cb1, Cb2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

Commit message: Final layout, electrical check OK, needs manual check
Parts:
- J11: symbol TERM-5 -> TERM-CPU
Connections:
- wire segments 102 -> 103
Changed lines of the file:
@@
 Text GLabel 2700 6200 0    45   Input ~ 0
 GND
-Text GLabel 3800 5800 2    45   Input ~ 0
+Text GLabel 4100 5800 2    45   Input ~ 0
 GND
 $Comp
@@
 NB: NT/GND pin\nused for EMI return ONLY\nNOT power return!
 $Comp
-L TERM-5 J11
+L TERM-CPU J11
 U 1 1 51C4790A
 P 8900 3850
@@
 	3400 5650 4200 5650
 Wire Wire Line
-	3800 5650 3800 5550
+	3800 5550 3800 5800
 Connection ~ 3800 5650
 Wire Wire Line
@@
 	6650 7000 6650 6800
 Wire Wire Line
-	6650 6800 6100 6800
-Wire Wire Line
-	6100 6800 6100 6400
+	6100 6800 6650 6800
+Wire Wire Line
+	6100 6400 6100 6800
 Wire Wire Line
 	6600 6500 6600 6650
@@
 Wire Wire Line
 	10700 1100 10700 1750
+Wire Wire Line
+	3800 5800 4100 5800
 $EndSCHEMATC

Commit message: Chnaged xtal caps to 22pf, fixed last board electrical checks
Parts:
- C19, C20: value 33pF -> 22pF
Changed lines of the file:
@@
 P 4150 2050
 F 0 "C19" H 4175 2100 30  0000 L CNN
-F 1 "33pF" H 4175 2000 30  0000 L CNN
+F 1 "22pF" H 4175 2000 30  0000 L CNN
 F 2 "~" H 4150 2050 60  0000 C CNN
 F 3 "~" H 4150 2050 60  0000 C CNN
@@
 P 4150 2450
 F 0 "C20" H 4175 2500 30  0000 L CNN
-F 1 "33pF" H 4175 2400 30  0000 L CNN
+F 1 "22pF" H 4175 2400 30  0000 L CNN
 F 2 "~" H 4150 2450 60  0000 C CNN
 F 3 "~" H 4150 2450 60  0000 C CNN

Commit message: Changes to make v3.3.2 boards
Added digital input protections, Vin protections, fixed footprints,
using right-angle headers on top of board for keypad/lcd.
Parts:
- removed D5: MUR410, symbol DIODESCH
- removed J10: ADC, symbol CONN_5
- removed J8: Scew terminals, symbol TERM-16
- removed R8, R9: 5k, symbol R2
- added C24: 0.1uF, symbol C
- added C25, C26, C27, C28: 4nF100V, symbol C
- added D10, D7: TVS-15V, symbol TVSX2
- added D6: TVS-13V, symbol TVS
- added D8, D9: STPS5L60, symbol DIODESCH
- added J10: ADC, symbol TERM-4
- added J12: STK, symbol TERM-4
- added J13: FLM, symbol TERM-4
- added J14: CC-Ser, symbol TERM-4
- added J15: LGHT, symbol TERM-2
- added J16: AUX, symbol TERM-4
- added J17: 12Vin, symbol TERM-2
- added J18: 5Vout, symbol TERM-2
- added R15, R18, R19, R20, R25, R31: 10k, symbol R2
- added R16, R21, R26, R32: 56.2k, symbol R2
- added R17, R22, R27, R33: 5k 2W PR, symbol R2
- added SW1, SW2: SW-DP3T, symbol SW-DP3T
- added TH1: PTC-3A, symbol THERMISTOR_SM
- added U6, U7: LM193, symbol LM193SM
- D1, D2, D3, D4: value MUR410 -> STPS5L60
- Q1, Q2, Q4: value RFD14N05 -> NTD5806NT4G
- Q3: value RFD14N05 -> BSS138K
- R2: value 10.2k -> 10k
- R7: value 5k -> 10k
- U2: value ATMEGA164PA-A -> ATMEGA324PA-A; symbol ATMEGA164PA-A -> ATMEGA324PA-A
- U3: value ACS755 -> ACS758
- U5: value V7805-2000 -> 5V-2A-PSU-V7805-2000
Connections:
- net labels added: +5Vout, 12Vin, AUX, AUXin, DRSNin, FLM+, FLM1in, FLM2in, Ip+, Ip-, NT-GND, PWR-IN, PWR-SW, Rx0-Ser, Rx0-TTL, Tx0-Ser, Tx0-TTL, Vref2.5
- net labels removed: AD3
- wire segments 103 -> 136
- no-connect marks 10 -> 14
Other:
- note added: "12 V Power entry & protection"
- note added: "12V UPS & 5V PSU"
- note added: "Baltimore Biodiesel BBD9000 SmartIO v3.3.2"
- note added: "Digital inputs"
- note added: "FLM+ select"
- note added: "Optional headers"
- note added: "Serial comms select"
- note removed: "12 V Power hold-up\nWith 5V 2A Sw. PSU\nV7805-2000"
- note removed: "3.3"
- note removed: "Baltimore Biodiesel BBD9000 SmartIO v3.3"
- note removed: "Optional ADC/DIO Hdr."
- note removed: "Power Rails"
- moved on the sheet: C10, C11, C12, C13, C14, C15, C16, C17, C21, C22, C23, C7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
