File: Kiosk/SmartIO/hardware/v3.3/SmartIOv3.3.sch (KiCad schematic (older format))
At the start: 98 parts, among them J1 LCD, J10 ADC, J11 TTL UART, J12 STK, J13 FLM, J14 CC-Ser, J15 LGHT, J16 AUX, J17 12Vin, J18 5Vout, J2 DB9, J3 MTN, J4 39910-0103, J6 ISP Hdr, J7 Keypad, K1 CB1aH-P-12V, Q1 NTD5806NT4G, Q2 NTD5806NT4G, Q3 BSS138K, Q4 NTD5806NT4G, Q5 BSS138K, Q6 BSS138K, SW1 SW-DP3T, SW2 SW-DP3T, U1 CPC1002N, U2 ATMEGA324PA-A, U3 ACS758, U4 MAX232, U5 5V-2A-PSU-V7805-2000, U6 LM193, U7 LM193, X1 18.432 MHz

Commit message: update universal FLM inputs in schematics (no board layout yet)
Parts:
- added Cb7, Cb8: 0.1uF, symbol C
- added R34, R35, R36, R37, R38, R39, R40, R41, R42, R43: 5k, symbol R2
- C25, C26, C27, C28: value 4nF100V -> 0.2uF 50V
- R15, R20, R25, R31: value 10k -> 5k
Connections:
- wire segments 136 -> 154
Other:
- moved on the sheet: C27, C28, J1, Q3, R15, R16, R17, R18, R19, R25, R26, R27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

Commit message: Finished layout for dig. inputs, incorporated footprint corrections
Parts:
- added H1, H2, H3, H4: Brd-Mnt, symbol HOLE
- added H10, H11, H7, H8, H9: Zip-Mnt, symbol HOLE
- added H5, H6: TCEHCBS, symbol HOLE
- added P1: LOGO-BBDC, symbol LOGO
- added P2: LOGO-OSHW, symbol LOGO
- U3: value ACS758 -> ACS758-050U; symbol ACS754_ACS755_ACS756_HALLCURRENTSENSOR -> ACS75X_CURRENT_SENSOR
Connections:
- net labels added: AUXin-C, DRSNin-C, FLM1in-C, FLM2in-C
Other:
- note added: "Logos &\nMounting Holes"
Changed lines of the file:
@@
 GND
 $Comp
-L ACS754_ACS755_ACS756_HALLCURRENTSENSOR U3
+L ACS75X_CURRENT_SENSOR U3
 U 1 1 51955960
 P 9100 2050
-F 0 "U3" H 8860 2200 60  0000 C CNN
-F 1 "ACS758" H 9220 2200 60  0000 C CNN
+F 0 "U3" H 8900 2000 60  0000 C CNN
+F 1 "ACS758-050U" H 9100 2200 60  0000 C CNN
 F 2 "" H 9100 2050 60  0001 C CNN
 F 3 "" H 9100 2050 60  0001 C CNN
@@
 NoConn ~ 9550 6850
 Text GLabel 9100 6450 2    45   Input ~ 0
+CCTx
+Text GLabel 9100 6650 2    45   Input ~ 0
 CCRx
-Text GLabel 9100 6650 2    45   Input ~ 0
-CCTx
 Text GLabel 7500 6550 0    45   Input ~ 0
 Rx0-Ser
@@
 V-TTL
 Text GLabel 7400 3200 0    45   Input ~ 0
+TTL-Tx
+Text GLabel 7400 3300 0    45   Input ~ 0
 TTL-Rx
-Text GLabel 7400 3300 0    45   Input ~ 0
-TTL-Tx
 Text GLabel 7400 3400 0    45   Input ~ 0
 +5V
@@
 $EndComp
 Text GLabel 8350 3500 0    45   Input ~ 0
-TTL-Tx
+TTL-Rx
 $Comp
 L R2 R12
@@
 $EndComp
 Text GLabel 8900 3500 2    45   Input ~ 0
-Tx0-TTL
+Rx0-TTL
 Text GLabel 8900 3100 2    45   Input ~ 0
 +5V
@@
 $EndComp
 Text GLabel 8350 4200 0    45   Input ~ 0
-TTL-Rx
+TTL-Tx
 $Comp
 L R2 R14
@@
 $EndComp
 Text GLabel 8900 4200 2    45   Input ~ 0
-Rx0-TTL
+Tx0-TTL
 Text GLabel 8900 3800 2    45   Input ~ 0
 +5V
@@
 +5V
 Text GLabel 1550 2500 0    45   Input ~ 0
+CCRx
+Text GLabel 1550 2400 0    45   Input ~ 0
 CCTx
-Text GLabel 1550 2400 0    45   Input ~ 0
-CCRx
 Text GLabel 1550 2600 0    45   Input ~ 0
 GND
@@
 $EndComp
 Connection ~ 2750 7400
+$Comp
+L LOGO P1
+U 1 1 52560D6E
+P 9700 4700
+F 0 "P1" H 9700 4700 30  0000 C CNN
+F 1 "LOGO-BBDC" H 9700 4600 30  0000 C CNN
+F 2 "" H 9700 4700 60  0000 C CNN
+F 3 "" H 9700 4700 60  0000 C CNN
+	1    9700 4700
+	1    0    0    -1
+$EndComp
+$Comp
+L LOGO P2
+U 1 1 52560E17
+P 9700 4500
+F 0 "P2" H 9700 4500 30  0000 C CNN
+F 1 "LOGO-OSHW" H 9700 4400 30  0000 C CNN
+F 2 "" H 9700 4500 60  0000 C CNN
+F 3 "" H 9700 4500 60  0000 C CNN
+	1    9700 4500
+	1    0    0    -1
+$EndComp
+$Comp
+L HOLE H1
+U 1 1 5256104B
+P 9950 4500
+F 0 "H1" H 9950 4500 30  0000 C CNN
+F 1 "Brd-Mnt" H 9950 4550 60  0001 C CNN
+F 2 "" H 9950 4500 60  0000 C CNN
+F 3 "" H 9950 4500 60  0000 C CNN
+	1    9950 4500
+	1    0    0    -1
+$EndComp
+$Comp
+L HOLE H2
+U 1 1 52561058
+P 10100 4500
+F 0 "H2" H 10100 4500 30  0000 C CNN
+F 1 "Brd-Mnt" H 10100 4550 60  0001 C CNN
+F 2 "" H 10100 4500 60  0000 C CNN
+F 3 "" H 10100 4500 60  0000 C CNN
+	1    10100 4500
+	1    0    0    -1
+$EndComp
+$Comp
+L HOLE H3
+U 1 1 5256105E
+P 9950 4650
+F 0 "H3" H 9950 4650 30  0000 C CNN
+F 1 "Brd-Mnt" H 9950 4700 60  0001 C CNN
+F 2 "" H 9950 4650 60  0000 C CNN
+F 3 "" H 9950 4650 60  0000 C CNN
+	1    9950 4650
+	1    0    0    -1
+$EndComp
+$Comp
+L HOLE H4
+U 1 1 52561064
+P 10100 4650
+F 0 "H4" H 10100 4650 30  0000 C CNN
+F 1 "Brd-Mnt" H 10100 4700 60  0001 C CNN
+F 2 "" H 10100 4650 60  0000 C CNN
+F 3 "" H 10100 4650 60  0000 C CNN
+	1    10100 4650
+	1    0    0    -1
+$EndComp
+Text Notes 9550 4300 0    60   ~ 0
+Logos &\nMounting Holes
+Text Label 2750 4350 0    25   ~ 0
+FLM1in-C
+Text Label 2750 5350 0    25   ~ 0
+FLM2in-C
+$Comp
+L HOLE H5
+U 1 1 52562E6D
+P 9950 4800
+F 0 "H5" H 9950 4800 30  0000 C CNN
+F 1 "TCEHCBS" H 9900 4700 30  0000 C CNN
+F 2 "" H 9950 4800 60  0000 C CNN
+F 3 "" H 9950 4800 60  0000 C CNN
+	1    9950 4800
+	1    0    0    -1
+$EndComp
+$Comp
+L HOLE H6
+U 1 1 52562E73
+P 10100 4800
+F 0 "H6" H 10100 4800 30  0000 C CNN
+F 1 "TCEHCBS" H 10150 4700 30  0000 C CNN
+F 2 "" H 10100 4800 60  0000 C CNN
+F 3 "" H 10100 4800 60  0000 C CNN
+	1    10100 4800
+	1    0    0    -1
+$EndComp
+$Comp
+L HOLE H7
+U 1 1 525631DA
+P 10250 4500
+F 0 "H7" H 10250 4500 30  0000 C CNN
+F 1 "Zip-Mnt" H 10250 4550 60  0001 C CNN
+F 2 "" H 10250 4500 60  0000 C CNN
+F 3 "" H 10250 4500 60  0000 C CNN
+	1    10250 4500
+	1    0    0    -1
+$EndComp
+$Comp
+L HOLE H8
+U 1 1 525631E0
+P 10400 4500
+F 0 "H8" H 10400 4500 30  0000 C CNN
+F 1 "Zip-Mnt" H 10400 4550 60  0001 C CNN
+F 2 "" H 10400 4500 60  0000 C CNN
+F 3 "" H 10400 4500 60  0000 C CNN
+	1    10400 4500
+	1    0    0    -1
+$EndComp
+$Comp
+L HOLE H9
+U 1 1 525631E6
+P 10250 4650
+F 0 "H9" H 10250 4650 30  0000 C CNN
+F 1 "Zip-Mnt" H 10250 4700 60  0001 C CNN
+F 2 "" H 10250 4650 60  0000 C CNN
+F 3 "" H 10250 4650 60  0000 C CNN
+	1    10250 4650
+	1    0    0    -1
+$EndComp
+$Comp
+L HOLE H10
+U 1 1 525631EC
+P 10400 4650
+F 0 "H10" H 10400 4650 30  0000 C CNN
+F 1 "Zip-Mnt" H 10400 4700 60  0001 C CNN
+F 2 "" H 10400 4650 60  0000 C CNN
+F 3 "" H 10400 4650 60  0000 C CNN
+	1    10400 4650
+	1    0    0    -1
+$EndComp
+$Comp
+L HOLE H11
+U 1 1 52563B38
+P 10400 4800
+F 0 "H11" H 10400 4800 30  0000 C CNN
+F 1 "Zip-Mnt" H 10400 4850 60  0001 C CNN
+F 2 "" H 10400 4800 60  0000 C CNN
+F 3 "" H 10400 4800 60  0000 C CNN
+	1    10400 4800
+	1    0    0    -1
+$EndComp
+Text Label 2700 6350 0    25   ~ 0
+AUXin-C
+Text Label 2750 7250 0    25   ~ 0
+DRSNin-C
 $EndSCHEMATC

Commit message: corrected ISP header-rows were mirorred
Other:
- note added: "Baltimore Biodiesel BBD9000 SmartIO v3.3.3"
- note removed: "Baltimore Biodiesel BBD9000 SmartIO v3.3.2"
- moved on the sheet: J6
Changed lines of the file:
@@
 L TERM-3X2 J6
 U 1 1 5190E361
-P 900 1850
-F 0 "J6" H 900 2100 50  0000 C CNN
-F 1 "ISP Hdr" V 900 1900 40  0000 C CNN
-F 2 "" H 900 1850 60  0001 C CNN
-F 3 "" H 900 1850 60  0001 C CNN
-	1    900  1850
+P 950 1800
+F 0 "J6" H 950 1650 50  0000 C CNN
+F 1 "ISP Hdr" V 950 1850 40  0000 C CNN
+F 2 "" H 950 1800 60  0001 C CNN
+F 3 "" H 950 1800 60  0001 C CNN
+	1    950  1800
 	1    0    0    -1
 $EndComp
@@
 	0    -1   -1   0
 $EndComp
-Text GLabel 1100 1900 2    45   Input ~ 0
+Text GLabel 750  1850 0    45   Input ~ 0
 ~RESET
-Text GLabel 1100 1800 2    45   Input ~ 0
+Text GLabel 750  1750 0    45   Input ~ 0
 PB7
 Text GLabel 1225 7725 2    45   Input ~ 0
@@
 Text GLabel 6650 3250 2    45   Input ~ 0
 PB6
-Text GLabel 1100 1700 2    45   Input ~ 0
+Text GLabel 750  1650 0    45   Input ~ 0
 PB6
-Text GLabel 700  1800 0    45   Input ~ 0
+Text GLabel 1150 1750 2    45   Input ~ 0
 PB5
 Text GLabel 1225 7525 2    45   Input ~ 0
@@
 Text GLabel 6650 2950 2    45   Input ~ 0
 PB3
-Text GLabel 700  1900 0    45   Input ~ 0
+Text GLabel 1150 1850 2    45   Input ~ 0
 GND
 Text Notes 7600 7600 0    60   ~ 0
-Baltimore Biodiesel BBD9000 SmartIO v3.3.2
+Baltimore Biodiesel BBD9000 SmartIO v3.3.3
 $Comp
 L MAX232 U4
@@
 Text GLabel 800  6150 0    45   Input ~ 0
 +12V
-Text GLabel 700  1700 0    45   Input ~ 0
+Text GLabel 1150 1650 2    45   Input ~ 0
 +5V
 Text GLabel 2750 3750 0    45   Input ~ 0

Commit message: Fixed reversed TTL Rx/Tx
Connections:
- no-connect marks 14 -> 18
Other:
- moved on the sheet: J11, Q5, Q6, R11, R12, R13, R14, SW1, SW2
Changed lines of the file:
@@
 L TERM-CPU J11
 U 1 1 51C4790A
-P 7800 3300
-F 0 "J11" V 7750 3300 50  0000 C CNN
-F 1 "TTL UART" V 7850 3300 50  0000 C CNN
-F 2 "" H 7800 3300 60  0000 C CNN
-F 3 "" H 7800 3300 60  0000 C CNN
-	1    7800 3300
-	1    0    0    -1
-$EndComp
-Text GLabel 7400 3100 0    45   Input ~ 0
+P 7600 3300
+F 0 "J11" V 7600 3350 50  0000 C CNN
+F 1 "TTL UART" V 7700 3350 50  0000 C CNN
+F 2 "" H 7600 3300 60  0000 C CNN
+F 3 "" H 7600 3300 60  0000 C CNN
+	1    7600 3300
+	1    0    0    -1
+$EndComp
+Text GLabel 7300 3350 0    45   Input ~ 0
 V-TTL
-Text GLabel 7400 3200 0    45   Input ~ 0
+Text GLabel 7300 3050 0    45   Input ~ 0
 TTL-Tx
-Text GLabel 7400 3300 0    45   Input ~ 0
+Text GLabel 7300 3150 0    45   Input ~ 0
 TTL-Rx
-Text GLabel 7400 3400 0    45   Input ~ 0
+Text GLabel 7300 3550 0    45   Input ~ 0
 +5V
-Text GLabel 7400 3500 0    45   Input ~ 0
+Text GLabel 7300 3450 0    45   Input ~ 0
 GND
 $Comp
 L MOSFET_N Q5
 U 1 1 51C47B69
-P 8700 3400
-F 0 "Q5" V 8500 3350 60  0000 R CNN
-F 1 "BSS138K" V 8900 3600 60  0000 R CNN
-F 2 "" H 8700 3400 60  0000 C CNN
-F 3 "" H 8700 3400 60  0000 C CNN
-	1    8700 3400
+P 8900 3400
+F 0 "Q5" V 8700 3350 60  0000 R CNN
+F 1 "BSS138K" V 9100 3600 60  0000 R CNN
+F 2 "" H 8900 3400 60  0000 C CNN
+F 3 "" H 8900 3400 60  0000 C CNN
+	1    8900 3400
 	0    1    1    0
 $EndComp
-Text GLabel 8350 3100 0    45   Input ~ 0
+Text GLabel 8550 3100 0    45   Input ~ 0
 V-TTL
 $Comp
 L R2 R11
 U 1 1 51C47BA6
-P 8450 3300
-F 0 "R11" V 8550 3500 50  0000 C CNN
-F 1 "10k" V 8450 3500 50  0000 C CNN
-F 2 "" H 8450 3300 60  0001 C CNN
-F 3 "" H 8450 3300 60  0001 C CNN
-	1    8450 3300
+P 8650 3300
+F 0 "R11" V 8750 3500 50  0000 C CNN
+F 1 "10k" V 8650 3500 50  0000 C CNN
+F 2 "" H 8650 3300 60  0001 C CNN
+F 3 "" H 8650 3300 60  0001 C CNN
+	1    8650 3300
 	0    -1   -1   0
 $EndComp
-Text GLabel 8350 3500 0    45   Input ~ 0
+Text GLabel 8550 3500 0    45   Input ~ 0
 TTL-Rx
 $Comp
 L R2 R12
 U 1 1 51C47CC6
-P 9000 3300
-F 0 "R12" V 9100 3300 50  0000 C CNN
-F 1 "10k" V 9000 3300 50  0000 C CNN
-F 2 "" H 9000 3300 60  0001 C CNN
-F 3 "" H 9000 3300 60  0001 C CNN
-	1    9000 3300
+P 9200 3300
+F 0 "R12" V 9300 3300 50  0000 C CNN
+F 1 "10k" V 9200 3300 50  0000 C CNN
+F 2 "" H 9200 3300 60  0001 C CNN
+F 3 "" H 9200 3300 60  0001 C CNN
+	1    9200 3300
 	0    -1   -1   0
 $EndComp
-Text GLabel 8900 3500 2    45   Input ~ 0
+Text GLabel 9100 3500 2    45   Input ~ 0
 Rx0-TTL
-Text GLabel 8900 3100 2    45   Input ~ 0
+Text GLabel 9100 3100 2    45   Input ~ 0
 +5V
 $Comp
@@
 L MOSFET_N Q6
 U 1 1 51C4CC9A
-P 8700 4100
-F 0 "Q6" V 8500 4050 60  0000 R CNN
-F 1 "BSS138K" V 8900 4300 60  0000 R CNN
-F 2 "" H 8700 4100 60  0000 C CNN
-F 3 "" H 8700 4100 60  0000 C CNN
-	1    8700 4100
+P 8900 4100
+F 0 "Q6" V 8700 4050 60  0000 R CNN
+F 1 "BSS138K" V 9100 4300 60  0000 R CNN
+F 2 "" H 8900 4100 60  0000 C CNN
+F 3 "" H 8900 4100 60  0000 C CNN
+	1    8900 4100
 	0    1    1    0
 $EndComp
-Text GLabel 8350 3800 0    45   Input ~ 0
+Text GLabel 8550 3800 0    45   Input ~ 0
 V-TTL
 $Comp
 L R2 R13
 U 1 1 51C4CCA1
-P 8450 4000
-F 0 "R13" V 8550 4200 50  0000 C CNN
-F 1 "10k" V 8450 4200 50  0000 C CNN
-F 2 "" H 8450 4000 60  0001 C CNN
-F 3 "" H 8450 4000 60  0001 C CNN
-	1    8450 4000
+P 8650 4000
+F 0 "R13" V 8750 4200 50  0000 C CNN
+F 1 "10k" V 8650 4200 50  0000 C CNN
+F 2 "" H 8650 4000 60  0001 C CNN
+F 3 "" H 8650 4000 60  0001 C CNN
+	1    8650 4000
 	0    -1   -1   0
 $EndComp
-Text GLabel 8350 4200 0    45   Input ~ 0
+Text GLabel 8550 4200 0    45   Input ~ 0
 TTL-Tx
 $Comp
 L R2 R14
 U 1 1 51C4CCA8
-P 9000 4000
-F 0 "R14" V 9100 4000 50  0000 C CNN
-F 1 "10k" V 9000 4000 50  0000 C CNN
-F 2 "" H 9000 4000 60  0001 C CNN
-F 3 "" H 9000 4000 60  0001 C CNN
-	1    9000 4000
+P 9200 4000
+F 0 "R14" V 9300 4000 50  0000 C CNN
+F 1 "10k" V 9200 4000 50  0000 C CNN
+F 2 "" H 9200 4000 60  0001 C CNN
+F 3 "" H 9200 4000 60  0001 C CNN
+	1    9200 4000
 	0    -1   -1   0
 $EndComp
-Text GLabel 8900 4200 2    45   Input ~ 0
+Text GLabel 9100 4200 2    45   Input ~ 0
 Tx0-TTL
-Text GLabel 8900 3800 2    45   Input ~ 0
+Text GLabel 9100 3800 2    45   Input ~ 0
 +5V
-Text Notes 7000 3000 0    60   ~ 0
+Text Notes 7700 2950 0    60   ~ 0
 TTL UART Voltage Conv.
 $Comp
@@
 Text GLabel 4100 1750 0    45   Input ~ 0
 GND
-Text Notes 7000 3700 0    60   ~ 0
+Text Notes 7100 3900 0    60   ~ 0
 Serial comms select
 $Comp
@@
 L SW-DP3T SW2
 U 1 1 51F6CE29
-P 9950 3400
-F 0 "SW2" H 9950 3050 40  0000 C CNN
-F 1 "SW-DP3T" H 9950 3750 40  0000 C CNN
-F 2 "" H 9700 3600 60  0000 C CNN
-F 3 "" H 9700 3600 60  0000 C CNN
-	1    9950 3400
-	1    0    0    -1
-$EndComp
-Text GLabel 9800 3150 0    45   Input ~ 0
+P 10000 3400
+F 0 "SW2" H 10000 3050 40  0000 C CNN
+F 1 "SW-DP3T" H 10000 3750 40  0000 C CNN
+F 2 "" H 9750 3600 60  0000 C CNN
+F 3 "" H 9750 3600 60  0000 C CNN
+	1    10000 3400
+	1    0    0    -1
+$EndComp
+Text GLabel 9850 3150 0    45   Input ~ 0
 +5Vout
-Text GLabel 9800 3650 0    45   Input ~ 0
+Text GLabel 9850 3650 0    45   Input ~ 0
 +12V
-Text Notes 9450 3000 0    60   ~ 0
+Text Notes 9500 3000 0    60   ~ 0
 FLM+ select
-Text GLabel 10150 3400 2    45   Input ~ 0
+Text GLabel 10200 3400 2    45   Input ~ 0
 FLM+
-NoConn ~ 9800 3250
-NoConn ~ 9800 3550
+NoConn ~ 9850 3250
+NoConn ~ 9850 3550
 $Comp
 L SW-DP3T SW1
 U 1 1 51F6F1A3
-P 7550 4100
-F 0 "SW1" H 7550 3750 40  0000 C CNN
-F 1 "SW-DP3T" H 7550 4450 40  0000 C CNN
-F 2 "" H 7300 4300 60  0000 C CNN
-F 3 "" H 7300 4300 60  0000 C CNN
-	1    7550 4100
-	1    0    0    -1
-$EndComp
-Text GLabel 7700 3950 2    45   Input ~ 0
+P 7650 4300
+F 0 "SW1" H 7650 3950 40  0000 C CNN
+F 1 "SW-DP3T" H 7650 4650 40  0000 C CNN
+F 2 "" H 7400 4500 60  0000 C CNN
+F 3 "" H 7400 4500 60  0000 C CNN
+	1    7650 4300
+	1    0    0    -1
+$EndComp
+Text GLabel 7800 4150 2    45   Input ~ 0
 Tx0
-Text GLabel 7700 4250 2    45   Input ~ 0
+Text GLabel 7800 4450 2    45   Input ~ 0
 Rx0
-Text GLabel 7400 3850 0    45   Input ~ 0
+Text GLabel 7500 4050 0    45   Input ~ 0
 Tx0-TTL
-Text GLabel 7400 4050 0    45   Input ~ 0
+Text GLabel 7500 4250 0    45   Input ~ 0
 Tx0-Ser
-Text GLabel 7400 4150 0    45   Input ~ 0
+Text GLabel 7500 4350 0    45   Input ~ 0
 Rx0-TTL
-Text GLabel 7400 4350 0    45   Input ~ 0
+Text GLabel 7500 4550 0    45   Input ~ 0
 Rx0-Ser
-NoConn ~ 7400 3950
-NoConn ~ 7400 4250
-Text GLabel 9800 3450 0    45   Input ~ 0
+NoConn ~ 7500 4150
+NoConn ~ 7500 4450
+Text GLabel 9850 3450 0    45   Input ~ 0
 +5Vout
-Text GLabel 9800 3350 0    45   Input ~ 0
+Text GLabel 9850 3350 0    45   Input ~ 0
 +12V
 Text Notes 550  3450 0    60   ~ 0
@@
 Connection ~ 5800 1350
 Wire Wire Line
-	8350 3500 8500 3500
-Wire Wire Line
-	8350 3100 8700 3100
-Wire Wire Line
-	8700 3100 8700 3200
+	8550 3500 8700 3500
+Wire Wire Line
+	8550 3100 8900 3100
+Wire Wire Line
+	8900 3100 8900 3200
 Wire Wire Line
 	6300 600  6300 1350
@@
 	9500 5250 9100 5250
 Wire Wire Line
-	8350 4200 8500 4200
-Wire Wire Line
-	8350 3800 8700 3800
-Wire Wire Line
-	8700 3800 8700 3900
+	8550 4200 8700 4200
+Wire Wire Line
+	8550 3800 8900 3800
+Wire Wire Line
+	8900 3800 8900 3900
 Wire Wire Line
 	9500 5850 9500 5650
@@
 Connection ~ 3150 1300
 Wire Wire Line
-	10100 3250 10100 3550
-Wire Wire Line
-	10150 3400 10100 3400
-Connection ~ 10100 3400
+	10150 3250 10150 3550
+Wire Wire Line
+	10200 3400 10150 3400
+Connection ~ 10150 3400
 Wire Wire Line
 	3550 6250 3550 6100
@@
 Text Label 2750 7250 0    25   ~ 0
 DRSNin-C
+Text GLabel 7300 3250 0    45   Input ~ 0
+GND
+Text GLabel 8000 3450 2    45   Input ~ 0
+GND
+Text GLabel 8000 3550 2    45   Input ~ 0
++5V
+NoConn ~ 8000 3350
+NoConn ~ 8000 3250
+NoConn ~ 8000 3150
+NoConn ~ 8000 3050
 $EndSCHEMATC

Commit message: Fixed olinuxino header pin#s & GND
Connections:
- no-connect marks 18 -> 16
Changed lines of the file:
@@
 Text GLabel 8000 3550 2    45   Input ~ 0
 +5V
-NoConn ~ 8000 3350
 NoConn ~ 8000 3250
-NoConn ~ 8000 3150
 NoConn ~ 8000 3050
+Text GLabel 8000 3150 2    45   Input ~ 0
+GND
+Text GLabel 8000 3350 2    45   Input ~ 0
+GND
 $EndSCHEMATC

Commit message: Fixed assy. spreadsheet and BOM to reflect 2.5V->3.3V Vref
Parts:
- R18: value 10k -> 5k
Connections:
- net labels added: Vref3.3
- net labels removed: Vref2.5
Changed lines of the file:
@@
-	-1   0    0    1
-$EndComp
-$Comp
-L R2 R18
-U 1 1 51F31F35
-P 3350 6150
-F 0 "R18" H 3300 6300 40  0000 C CNN
-F 1 "10k" H 3450 6300 40  0000 C CNN
-F 2 "" H 3350 6150 60  0001 C CNN
-F 3 "" H 3350 6150 60  0001 C CNN
-	1    3350 6150
 	-1   0    0    1
 $EndComp
@@
 AUX
 Text GLabel 3550 6100 2    45   Input ~ 0
-Vref2.5
+Vref3.3
 Text GLabel 3350 7850 0    45   Input ~ 0
-Vref2.5
+Vref3.3
 Text GLabel 3350 6950 0    45   Input ~ 0
-Vref2.5
+Vref3.3
 $Comp
 L C C27
@@
 Text GLabel 8000 3350 2    45   Input ~ 0
 GND
+$Comp
+L R2 R18
+U 1 1 5292EC73
+P 3350 6150
+F 0 "R18" H 3250 6300 40  0000 C CNN
+F 1 "5k" H 3400 6300 40  0000 C CNN
+F 2 "" H 3350 6150 60  0001 C CNN
+F 3 "" H 3350 6150 60  0001 C CNN
+	1    3350 6150
+	-1   0    0    1
+$EndComp
 $EndSCHEMATC
