File: Kiosk/SmartIO/hardware/v3.3/SmartIOv3.3.sch (KiCad schematic (older format))
At the start: 123 parts, among them J1 LCD, J10 ADC, J11 TTL UART, J12 STK, J13 FLM, J14 CC-Ser, J15 LGHT, J16 AUX, J17 12Vin, J18 5Vout, J2 DB9, J3 MTN, J4 39910-0103, J6 ISP Hdr, J7 Keypad, K1 CB1aH-P-12V, P1 LOGO-BBDC, P2 LOGO-OSHW, Q1 NTD5806NT4G, Q2 NTD5806NT4G, Q3 BSS138K, Q4 NTD5806NT4G, Q5 BSS138K, Q6 BSS138K, SW1 SW-DP3T, SW2 SW-DP3T, U1 CPC1002N, U2 ATMEGA324PA-A, U3 ACS758-050U, U4 MAX232, U5 5V-2A-PSU-V7805-2000, U6 LM193, U7 LM193, X1 18.432 MHz

Commit message: Added UPS charge current limiter, U7 on +5Vout
Simple current limiter using two 75 ohm 3W resistors in parallel with a
diode - charging through 37.5 ohm/6W, discharge through diode.
Parts:
- added D11: STPS5L60, symbol DIODESCH
- added R44, R45: 75 3W, symbol R2
Connections:
- wire segments 154 -> 157
Other:
- moved on the sheet: C12, C13, C14, C15, C16, C17, C22, C23, D8, D9, U5
Changed lines of the file:
@@
 L CP1 C12
 U 1 1 5197970E
-P 2750 2550
-F 0 "C12" H 2480 2580 40  0000 L CNN
-F 1 "10F" H 2490 2490 40  0000 L CNN
-F 2 "" H 2750 2550 60  0001 C CNN
-F 3 "" H 2750 2550 60  0001 C CNN
-	1    2750 2550
+P 2750 2850
+F 0 "C12" H 2480 2880 40  0000 L CNN
+F 1 "10F" H 2490 2790 40  0000 L CNN
+F 2 "" H 2750 2850 60  0001 C CNN
+F 3 "" H 2750 2850 60  0001 C CNN
+	1    2750 2850
 	1    0    0    -1
 $EndComp
@@
 L CP1 C13
 U 1 1 51979879
-P 2750 2950
-F 0 "C13" H 2490 3020 40  0000 L CNN
-F 1 "10F" H 2500 2940 40  0000 L CNN
-F 2 "" H 2750 2950 60  0001 C CNN
-F 3 "" H 2750 2950 60  0001 C CNN
-	1    2750 2950
+P 2750 3250
+F 0 "C13" H 2490 3320 40  0000 L CNN
+F 1 "10F" H 2500 3240 40  0000 L CNN
+F 2 "" H 2750 3250 60  0001 C CNN
+F 3 "" H 2750 3250 60  0001 C CNN
+	1    2750 3250
 	1    0    0    -1
 $EndComp
@@
 L CP1 C14
 U 1 1 51979886
-P 2750 3350
-F 0 "C14" H 2490 3410 40  0000 L CNN
-F 1 "10F" H 2500 3330 40  0000 L CNN
-F 2 "" H 2750 3350 60  0001 C CNN
-F 3 "" H 2750 3350 60  0001 C CNN
-	1    2750 3350
+P 2750 3650
+F 0 "C14" H 2490 3710 40  0000 L CNN
+F 1 "10F" H 2500 3630 40  0000 L CNN
+F 2 "" H 2750 3650 60  0001 C CNN
+F 3 "" H 2750 3650 60  0001 C CNN
+	1    2750 3650
 	1    0    0    -1
 $EndComp
@@
 L CP1 C15
 U 1 1 5197988C
-P 3150 3350
-F 0 "C15" H 2880 3290 40  0000 L CNN
-F 1 "10F" H 2880 3390 40  0000 L CNN
-F 2 "" H 3150 3350 60  0001 C CNN
-F 3 "" H 3150 3350 60  0001 C CNN
-	1    3150 3350
+P 3150 3650
+F 0 "C15" H 2880 3590 40  0000 L CNN
+F 1 "10F" H 2880 3690 40  0000 L CNN
+F 2 "" H 3150 3650 60  0001 C CNN
+F 3 "" H 3150 3650 60  0001 C CNN
+	1    3150 3650
 	-1   0    0    1
 $EndComp
@@
 L CP1 C16
 U 1 1 5197989C
-P 3150 2950
-F 0 "C16" H 2890 2870 40  0000 L CNN
-F 1 "10F" H 2890 2960 40  0000 L CNN
-F 2 "" H 3150 2950 60  0001 C CNN
-F 3 "" H 3150 2950 60  0001 C CNN
-	1    3150 2950
+P 3150 3250
+F 0 "C16" H 2890 3170 40  0000 L CNN
+F 1 "10F" H 2890 3260 40  0000 L CNN
+F 2 "" H 3150 3250 60  0001 C CNN
+F 3 "" H 3150 3250 60  0001 C CNN
+	1    3150 3250
 	-1   0    0    1
 $EndComp
@@
 L CP1 C17
 U 1 1 519798A2
-P 3150 2550
-F 0 "C17" H 2890 2500 40  0000 L CNN
-F 1 "10F" H 2890 2590 40  0000 L CNN
-F 2 "" H 3150 2550 60  0001 C CNN
-F 3 "" H 3150 2550 60  0001 C CNN
-	1    3150 2550
+P 3150 2850
+F 0 "C17" H 2890 2800 40  0000 L CNN
+F 1 "10F" H 2890 2890 40  0000 L CNN
+F 2 "" H 3150 2850 60  0001 C CNN
+F 3 "" H 3150 2850 60  0001 C CNN
+	1    3150 2850
 	-1   0    0    1
 $EndComp
@@
 Text GLabel 5650 5450 2    45   Input ~ 0
 GND
-Text GLabel 3450 2350 2    45   Input ~ 0
+Text GLabel 3450 2250 2    45   Input ~ 0
 GND
 $Comp
@@
 Text Notes 7610 720  0    60   ~ 0
 Power Relay, Drive (PA7) and Current Sense (PA1)\nIsolated PWR, NT/GND. 12VDC/120VAC.
-Text Notes 1900 1550 0    60   ~ 0
+Text Notes 1850 1600 0    60   ~ 0
 12V UPS & 5V PSU
 Text Notes 7400 5000 0    60   ~ 0
@@
 L LM7805 U5
 U 1 1 51C25E9D
-P 3150 1850
-F 0 "U5" H 3300 1654 60  0000 C CNN
-F 1 "5V-2A-PSU-V7805-2000" H 3150 2050 40  0000 C CNN
-F 2 "" H 3150 1850 60  0000 C CNN
-F 3 "" H 3150 1850 60  0000 C CNN
-	1    3150 1850
+P 3150 1750
+F 0 "U5" H 3300 1554 60  0000 C CNN
+F 1 "5V-2A-PSU-V7805-2000" H 3350 1950 40  0000 C CNN
+F 2 "" H 3150 1750 60  0000 C CNN
+F 3 "" H 3150 1750 60  0000 C CNN
+	1    3150 1750
 	1    0    0    -1
 $EndComp
@@
 L C C23
 U 1 1 51C25ECB
-P 3550 2000
-F 0 "C23" V 3570 2120 40  0000 C TNN
-F 1 "22uF" V 3590 1810 39  0000 L CNN
-F 2 "" H 3550 2000 60  0001 C CNN
-F 3 "" H 3550 2000 60  0001 C CNN
-	1    3550 2000
+P 3550 1900
+F 0 "C23" V 3570 2020 40  0000 C TNN
+F 1 "22uF" V 3590 1710 39  0000 L CNN
+F 2 "" H 3550 1900 60  0001 C CNN
+F 3 "" H 3550 1900 60  0001 C CNN
+	1    3550 1900
 	-1   0    0    1
 $EndComp
@@
 L C C22
 U 1 1 51C25ED1
-P 2750 2000
-F 0 "C22" V 2770 2120 40  0000 C TNN
-F 1 "10uF" V 2790 1810 39  0000 L CNN
-F 2 "" H 2750 2000 60  0001 C CNN
-F 3 "" H 2750 2000 60  0001 C CNN
-	1    2750 2000
-	-1   0    0    1
-$EndComp
-Text GLabel 3550 1800 2    45   Input ~ 0
+P 2750 1900
+F 0 "C22" V 2770 2020 40  0000 C TNN
+F 1 "10uF" V 2790 1710 39  0000 L CNN
+F 2 "" H 2750 1900 60  0001 C CNN
+F 3 "" H 2750 1900 60  0001 C CNN
+	1    2750 1900
+	-1   0    0    1
+$EndComp
+Text GLabel 3550 1700 2    45   Input ~ 0
 +5V
 Text Notes 9150 970  0    39   ~ 0
@@
 GND
 Text GLabel 4250 7400 2    45   Input ~ 0
-+5V
++5Vout
 $Comp
 L R2 R25
@@
 GND
 Text GLabel 4250 6500 2    45   Input ~ 0
-+5V
++5Vout
 $Comp
 L R2 R31
@@
 Text GLabel 3850 6850 2    45   Input ~ 0
 AUX
-Text GLabel 2050 1850 2    45   Input ~ 0
+Text GLabel 2050 1750 2    45   Input ~ 0
 +12V
 $Comp
 L DIODESCH D8
 U 1 1 51F6B6D6
-P 2250 2150
-F 0 "D8" H 2150 2325 40  0000 C CNN
-F 1 "STPS5L60" H 2250 2250 40  0000 C CNN
-F 2 "" H 2250 2150 60  0001 C CNN
-F 3 "" H 2250 2150 60  0001 C CNN
-	1    2250 2150
+P 2250 2050
+F 0 "D8" H 2150 2225 40  0000 C CNN
+F 1 "STPS5L60" H 2250 2150 40  0000 C CNN
+F 2 "" H 2250 2050 60  0001 C CNN
+F 3 "" H 2250 2050 60  0001 C CNN
+	1    2250 2050
 	1    0    0    -1
 $EndComp
@@
 Text GLabel 1150 1650 2    45   Input ~ 0
 +5V
-Text GLabel 2750 3750 0    45   Input ~ 0
+Text GLabel 3950 3650 0    45   Input ~ 0
 +5V
 $Comp
 L DIODESCH D9
 U 1 1 51F6C8A3
-P 2950 3750
-F 0 "D9" H 2800 3850 40  0000 C CNN
-F 1 "STPS5L60" H 3000 3850 40  0000 C CNN
-F 2 "" H 2950 3750 60  0001 C CNN
-F 3 "" H 2950 3750 60  0001 C CNN
-	1    2950 3750
-	1    0    0    -1
-$EndComp
-Text GLabel 3150 3750 2    45   Input ~ 0
+P 4150 3650
+F 0 "D9" H 4000 3750 40  0000 C CNN
+F 1 "STPS5L60" H 4200 3750 40  0000 C CNN
+F 2 "" H 4150 3650 60  0001 C CNN
+F 3 "" H 4150 3650 60  0001 C CNN
+	1    4150 3650
+	1    0    0    -1
+$EndComp
+Text GLabel 4350 3650 2    45   Input ~ 0
 +5Vout
 $Comp
@@
 	800  6650 1000 6650
 Wire Wire Line
-	2450 2350 2750 2350
-Wire Wire Line
-	2750 2200 3550 2200
-Wire Wire Line
-	3150 2100 3150 2350
-Connection ~ 3150 2200
-Wire Wire Line
-	2750 3550 3150 3550
+	2450 2175 2750 2175
+Wire Wire Line
+	2750 2100 3550 2100
+Wire Wire Line
+	3150 2000 3150 2650
+Connection ~ 3150 2100
+Wire Wire Line
+	2750 3850 3150 3850
 Wire Wire Line
 	8850 1400 8500 1400
@@
 	6475 5925 6475 6575
 Wire Wire Line
-	3150 2350 3450 2350
+	3150 2250 3450 2250
 Wire Wire Line
 	2350 1000 2350 1300
@@
 	800  4350 800  4450
 Wire Wire Line
-	3550 1800 3550 1800
+	3550 1700 3550 1700
 Connection ~ 3150 1300
 Wire Wire Line
@@
 	3150 800  3150 900
 Wire Wire Line
-	2750 1800 2450 1800
-Wire Wire Line
-	2450 1800 2450 2350
-Connection ~ 2450 2150
-Wire Wire Line
-	2050 1850 2050 2150
+	2750 1700 2450 1700
+Wire Wire Line
+	2450 1700 2450 2175
+Connection ~ 2450 2050
+Wire Wire Line
+	2050 1750 2050 2050
 Wire Wire Line
 	3150 900  2750 900
@@
 L PWR_FLAG #FLG09
 U 1 1 52362F4A
-P 3150 3750
-F 0 "#FLG09" H 3150 3845 30  0001 C CNN
-F 1 "PWR_FLAG" H 3150 3930 30  0000 C CNN
-F 2 "" H 3150 3750 60  0001 C CNN
-F 3 "" H 3150 3750 60  0001 C CNN
-	1    3150 3750
+P 4350 3650
+F 0 "#FLG09" H 4350 3745 30  0001 C CNN
+F 1 "PWR_FLAG" H 4350 3830 30  0000 C CNN
+F 2 "" H 4350 3650 60  0001 C CNN
+F 3 "" H 4350 3650 60  0001 C CNN
+	1    4350 3650
 	-1   0    0    1
 $EndComp
@@
 	-1   0    0    1
 $EndComp
+$Comp
+L R2 R44
+U 1 1 52AA4B14
+P 2950 2450
+F 0 "R44" H 2825 2475 40  0000 C CNN
+F 1 "75 3W" H 3025 2475 40  0000 C CNN
+F 2 "" H 2950 2450 60  0001 C CNN
+F 3 "" H 2950 2450 60  0001 C CNN
+	1    2950 2450
+	0    -1   -1   0
+$EndComp
+$Comp
+L DIODESCH D11
+U 1 1 52AA4B22
+P 2450 2450
+F 0 "D11" H 2350 2625 40  0000 C CNN
+F 1 "STPS5L60" H 2450 2550 40  0000 C CNN
+F 2 "" H 2450 2450 60  0001 C CNN
+F 3 "" H 2450 2450 60  0001 C CNN
+	1    2450 2450
+	0    -1   -1   0
+$EndComp
+Wire Wire Line
+	2450 2650 2850 2650
+Connection ~ 2750 2650
+Wire Wire Line
+	2450 2250 2850 2250
+Wire Wire Line
+	2750 2175 2750 2250
+Connection ~ 2750 2250
+Connection ~ 3150 2250
+$Comp
+L R2 R45
+U 1 1 52AB8C2B
+P 2700 2450
+F 0 "R45" H 2575 2475 40  0000 C CNN
+F 1 "75 3W" H 2775 2475 40  0000 C CNN
+F 2 "" H 2700 2450 60  0001 C CNN
+F 3 "" H 2700 2450 60  0001 C CNN
+	1    2700 2450
+	0    -1   -1   0
+$EndComp
+Connection ~ 2600 2250
+Connection ~ 2600 2650
+Connection ~ 2850 2250
+Connection ~ 2850 2650
 $EndSCHEMATC

Commit message: Fixed case in components for latest eeschema
Parts:
- C19, C20: symbol CSMALL -> Csmall
- D10, D7: symbol TVSX2 -> TVSx2
- U3: symbol ACS75X_CURRENT_SENSOR -> ACS75x_CURRENT_SENSOR
- U6, U7: symbol LM193SM -> LM193sm
Changed lines of the file:
@@
 EESchema Schematic File Version 2
+LIBS:components
+LIBS:connectors
+LIBS:SmartIOv3.3-cache
 LIBS:power
 LIBS:device
@@
 LIBS:valves
 LIBS:SmartIOv3.3-cache
-LIBS:connectors
-LIBS:components
-LIBS:SmartIOv3.3-cache
 EELAYER 24 0
 EELAYER END
@@
 GND
 $Comp
-L ACS75X_CURRENT_SENSOR U3
+L ACS75x_CURRENT_SENSOR U3
 U 1 1 51955960
 P 9100 2050
@@
 Screw Terminals
 $Comp
-L CSMALL C19
+L Csmall C19
 U 1 1 5197ECE5
 P 4150 2050
@@
 $EndComp
 $Comp
-L CSMALL C20
+L Csmall C20
 U 1 1 5197ED13
 P 4150 2450
@@
 ~RESET
 $Comp
-L LM193SM U6
+L LM193sm U6
 U 1 1 51F31B63
 P 3650 4600
@@
 FLM1in
 $Comp
-L TVSX2 D7
+L TVSx2 D7
 U 1 1 51F3204F
 P 2600 4700
@@
 FLM1
 $Comp
-L LM193SM U7
+L LM193sm U7
 U 2 1 51F32D25
 P 3650 7750
@@
 DRSN
 $Comp
-L LM193SM U7
+L LM193sm U7
 U 1 1 51F32CF0
 P 3650 6850
@@
 $EndComp
 $Comp
-L TVSX2 D10
+L TVSx2 D10
 U 1 1 51F80F47
 P 2750 7600
@@
 $EndComp
 $Comp
-L TVSX2 D10
+L TVSx2 D10
 U 2 1 51F80F56
 P 2700 6700
@@
 	2200 4250 2350 4250
 $Comp
-L LM193SM U6
+L LM193sm U6
 U 2 1 523631BE
 P 3650 5550
@@
 FLM2in
 $Comp
-L TVSX2 D7
+L TVSx2 D7
 U 2 1 523631D8
 P 2600 5650
